File: Bluetooth.kicad_sch (KiCad schematic)
At the start: 2 parts

Commit message: Merged in everyone's schematic changes
Parts:
- added D10, D11: D_Small, symbol Device:D_Small
- added R? (x2): 1k, symbol Device:R_Small
- gave numbers to parts that had none: 2
Connections:
- net GND: now also R?.1, R?.2
- net RX: now also D10.2 (A)
- net TX: now also D11.2 (A)
- new net: D10.1 (K), R?.1
- new net: D11.1 (K), R?.2
Other:
- note added: "Bluetooth"
- moved on the sheet: J50, R40
Changed lines of the file:
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@@
 (kicad_sch (version 20211123) (generator eeschema)
   (paper "A4")
-  (no_connect (at 82.55 69.85))
-  (no_connect (at 82.55 57.15))
-  (wire (pts (xy 88.9 67.31) (xy 82.55 67.31))
+  (junction (at 24.13 52.07) (diameter 0) (color 0 0 0 0)
+  )
+  (no_connect (at 34.29 41.275))
+  (no_connect (at 34.29 28.575))
+  (wire (pts (xy 24.13 52.07) (xy 24.13 52.705))
     (stroke (width 0) (type default) (color 0 0 0 0))
   )
-  (wire (pts (xy 82.55 59.69) (xy 101.6 59.69))
+  (wire (pts (xy 33.655 49.53) (xy 40.64 49.53))
     (stroke (width 0) (type default) (color 0 0 0 0))
   )
-  (wire (pts (xy 82.55 62.23) (xy 101.6 62.23))
+  (wire (pts (xy 40.64 38.735) (xy 34.29 38.735))
     (stroke (width 0) (type default) (color 0 0 0 0))
   )
-  (global_label "TX" (shape input) (at 93.98 67.31 0) (fields_autoplaced)
+  (wire (pts (xy 45.72 52.07) (xy 50.8 52.07))
+    (stroke (width 0) (type default) (color 0 0 0 0))
+  )
+  (wire (pts (xy 33.655 52.07) (xy 40.64 52.07))
+    (stroke (width 0) (type default) (color 0 0 0 0))
+  )
+  (wire (pts (xy 28.575 49.53) (xy 24.13 49.53))
+    (stroke (width 0) (type default) (color 0 0 0 0))
+  )
+  (wire (pts (xy 28.575 52.07) (xy 24.13 52.07))
+    (stroke (width 0) (type default) (color 0 0 0 0))
+  )
+  (wire (pts (xy 45.72 49.53) (xy 50.8 49.53))
+    (stroke (width 0) (type default) (color 0 0 0 0))
+  )
+  (wire (pts (xy 34.29 31.115) (xy 53.34 31.115))
+    (stroke (width 0) (type default) (color 0 0 0 0))
+  )
+  (wire (pts (xy 24.13 49.53) (xy 24.13 52.07))
+    (stroke (width 0) (type default) (color 0 0 0 0))
+  )
+  (wire (pts (xy 34.29 33.655) (xy 53.34 33.655))
+    (stroke (width 0) (type default) (color 0 0 0 0))
+  )
+  (text "Bluetooth" (at 35.56 22.86 0)
+    (effects (font (size 1.27 1.27)) (justify left bottom))
+  )
+  (global_label "TX" (shape input) (at 45.72 38.735 0) (fields_autoplaced)
     (effects (font (size 1.27 1.27)) (justify left))
-    (property "Intersheet References" "${INTERSHEET_REFS}" (id 0) (at 98.5702 67.3894 0)
+    (property "Intersheet References" "${INTERSHEET_REFS}" (id 0) (at 50.3102 38.8144 0)
       (effects (font (size 1.27 1.27)) (justify left) hide)
     )
   )
-  (global_label "RX" (shape input) (at 82.55 64.77 0) (fields_autoplaced)
+  (global_label "RX" (shape input) (at 50.8 49.53 0) (fields_autoplaced)
     (effects (font (size 1.27 1.27)) (justify left))
-    (property "Intersheet References" "${INTERSHEET_REFS}" (id 0) (at 87.4426 64.8494 0)
+    (property "Intersheet References" "${INTERSHEET_REFS}" (id 0) (at 55.6926 49.4506 0)
       (effects (font (size 1.27 1.27)) (justify left) hide)
     )
   )
-  (symbol (lib_id "power:+5V") (at 101.6 59.69 0) (unit 1)
-    (in_bom yes) (on_board yes) (fields_autoplaced)
-    (property "Reference" "#PWR?" (id 0) (at 101.6 63.5 0)
+  (global_label "RX" (shape input) (at 34.29 36.195 0) (fields_autoplaced)
+    (effects (font (size 1.27 1.27)) (justify left))
+    (property "Intersheet References" "${INTERSHEET_REFS}" (id 0) (at 39.1826 36.2744 0)
+      (effects (font (size 1.27 1.27)) (justify left) hide)
+    )
+  )
+  (global_label "TX" (shape input) (at 50.8 52.07 0) (fields_autoplaced)
+    (effects (font (size 1.27 1.27)) (justify left))
+    (property "Intersheet References" "${INTERSHEET_REFS}" (id 0) (at 55.3902 51.9906 0)
+      (effects (font (size 1.27 1.27)) (justify left) hide)
+    )
+  )
+  (symbol (lib_id "Device:R_Small") (at 31.115 49.53 270) (unit 1)
+    (in_bom yes) (on_board yes)
+    (property "Reference" "R?" (id 0) (at 31.115 47.625 90))
+    (property "Value" "1k" (id 1) (at 31.115 45.72 90))
+    (property "Footprint" "" (id 2) (at 31.115 49.53 0)
       (effects (font (size 1.27 1.27)) hide)
     )
-    (property "Value" "+5V" (id 1) (at 101.6 56.1142 0))
-    (property "Footprint" "" (id 2) (at 101.6 59.69 0)
+    (property "Datasheet" "~" (id 3) (at 31.115 49.53 0)
       (effects (font (size 1.27 1.27)) hide)
     )
-    (property "Datasheet" "" (id 3) (at 101.6 59.69 0)
+    (pin "1")
+    (pin "2")
+  )
+  (symbol (lib_id "power:+5V") (at 53.34 31.115 0) (unit 1)
+    (in_bom yes) (on_board yes) (fields_autoplaced)
+    (property "Reference" "#PWR?" (id 0) (at 53.34 34.925 0)
+      (effects (font (size 1.27 1.27)) hide)
+    )
+    (property "Value" "+5V" (id 1) (at 53.34 27.5392 0))
+    (property "Footprint" "" (id 2) (at 53.34 31.115 0)
+      (effects (font (size 1.27 1.27)) hide)
+    )
+    (property "Datasheet" "" (id 3) (at 53.34 31.115 0)
       (effects (font (size 1.27 1.27)) hide)
     )
     (pin "1")
   )
-  (symbol (lib_id "CustomSymbols:HC-05") (at 82.55 63.5 270) (unit 1)
+  (symbol (lib_id "CustomSymbols:HC-05") (at 34.29 34.925 270) (unit 1)
     (in_bom yes) (on_board yes) (fields_autoplaced)
-    (property "Reference" "J?" (id 0) (at 72.9488 64.3347 90)
-      (effects (font (size 1.27 1.27)) (justify right))
-    )
-    (property "Value" "HC-05" (id 1) (at 72.9488 61.7978 90)
-      (effects (font (size 1.27 1.27)) (justify right))
-    )
-    (property "Footprint" "" (id 2) (at 82.55 58.42 0)
+    (property "Reference" "J50" (id 0) (at 28.575 23.656 90))
+    (property "Value" "HC-05" (id 1) (at 28.575 26.1929 90))
+    (property "Footprint" "" (id 2) (at 34.29 29.845 0)
       (effects (font (size 1.27 1.27)) hide)
     )
-    (property "Datasheet" "" (id 3) (at 82.55 58.42 0)
+    (property "Datasheet" "" (id 3) (at 34.29 29.845 0)
       (effects (font (size 1.27 1.27)) hide)
     )
@@
     (pin "6")
   )
-  (symbol (lib_id "Device:R_Small") (at 91.44 67.31 270) (unit 1)
-    (in_bom yes) (on_board yes) (fields_autoplaced)
-    (property "Reference" "R?" (id 0) (at 91.44 71.7464 90))
-    (property "Value" "100r" (id 1) (at 91.44 69.2095 90))
-    (property "Footprint" "" (id 2) (at 91.44 67.31 0)
+  (symbol (lib_id "Device:D_Small") (at 43.18 52.07 0) (unit 1)
+    (in_bom yes) (on_board yes)
+    (property "Reference" "D11" (id 0) (at 43.18 54.61 0))
+    (property "Value" "D_Small" (id 1) (at 43.18 56.515 0))
+    (property "Footprint" "" (id 2) (at 43.18 52.07 90)
       (effects (font (size 1.27 1.27)) hide)
     )
-    (property "Datasheet" "~" (id 3) (at 91.44 67.31 0)
+    (property "Datasheet" "~" (id 3) (at 43.18 52.07 90)
       (effects (font (size 1.27 1.27)) hide)
     )
@@
     (pin "2")
   )
-  (symbol (lib_id "power:GND") (at 101.6 62.23 0) (unit 1)
-    (in_bom yes) (on_board yes) (fields_autoplaced)
-    (property "Reference" "#PWR?" (id 0) (at 101.6 68.58 0)
+  (symbol (lib_id "Device:R_Small") (at 43.18 38.735 270) (unit 1)
+    (in_bom yes) (on_board yes)
+    (property "Reference" "R40" (id 0) (at 43.18 40.64 90))
+    (property "Value" "100r" (id 1) (at 43.18 36.8355 90))
+    (property "Footprint" "" (id 2) (at 43.18 38.735 0)
       (effects (font (size 1.27 1.27)) hide)
     )
-    (property "Value" "GND" (id 1) (at 101.6 66.6734 0))
-    (property "Footprint" "" (id 2) (at 101.6 62.23 0)
+    (property "Datasheet" "~" (id 3) (at 43.18 38.735 0)
       (effects (font (size 1.27 1.27)) hide)
     )
-    (property "Datasheet" "" (id 3) (at 101.6 62.23 0)
+    (pin "1")
+    (pin "2")
+  )
+  (symbol (lib_id "power:GND") (at 24.13 52.705 0) (unit 1)
+    (in_bom yes) (on_board yes) (fields_autoplaced)
+    (property "Reference" "#PWR?" (id 0) (at 24.13 59.055 0)
+      (effects (font (size 1.27 1.27)) hide)
+    )
+    (property "Value" "GND" (id 1) (at 24.13 57.1484 0))
+    (property "Footprint" "" (id 2) (at 24.13 52.705 0)
+      (effects (font (size 1.27 1.27)) hide)
+    )
+    (property "Datasheet" "" (id 3) (at 24.13 52.705 0)
       (effects (font (size 1.27 1.27)) hide)
     )
     (pin "1")
   )
+  (symbol (lib_id "Device:D_Small") (at 43.18 49.53 0) (unit 1)
+    (in_bom yes) (on_board yes)
+    (property "Reference" "D10" (id 0) (at 43.18 45.72 0))
+    (property "Value" "D_Small" (id 1) (at 43.18 47.3511 0))
+    (property "Footprint" "" (id 2) (at 43.18 49.53 90)
+      (effects (font (size 1.27 1.27)) hide)
+    )
+    (property "Datasheet" "~" (id 3) (at 43.18 49.53 90)
+      (effects (font (size 1.27 1.27)) hide)
+    )
+    (pin "1")
+    (pin "2")
+  )
+  (symbol (lib_id "power:GND") (at 53.34 33.655 0) (unit 1)
+    (in_bom yes) (on_board yes) (fields_autoplaced)
+    (property "Reference" "#PWR?" (id 0) (at 53.34 40.005 0)
+      (effects (font (size 1.27 1.27)) hide)
+    )
+    (property "Value" "GND" (id 1) (at 53.34 38.0984 0))
+    (property "Footprint" "" (id 2) (at 53.34 33.655 0)
+      (effects (font (size 1.27 1.27)) hide)
+    )
+    (property "Datasheet" "" (id 3) (at 53.34 33.655 0)
+      (effects (font (size 1.27 1.27)) hide)
+    )
+    (pin "1")
+  )
+  (symbol (lib_id "Device:R_Small") (at 31.115 52.07 90) (unit 1)
+    (in_bom yes) (on_board yes)
+    (property "Reference" "R?" (id 0) (at 31.115 53.975 90))
+    (property "Value" "1k" (id 1) (at 31.115 55.88 90))
+    (property "Footprint" "" (id 2) (at 31.115 52.07 0)
+      (effects (font (size 1.27 1.27)) hide)
+    )
+    (property "Datasheet" "~" (id 3) (at 31.115 52.07 0)
+      (effects (font (size 1.27 1.27)) hide)
+    )
+    (pin "1")
+    (pin "2")
+  )
 )

Commit message: Finishing touches (associating footprints) to schematic
Parts:
- removed D10, D11: D_Small, symbol Device:D_Small
- added D10, D11: LED_Small, Diode_SMD:D_0805_2012Metric, symbol Device:LED_Small
- J50: footprint (none) -> CustomFootprints:HC-05
- R40: footprint (none) -> Resistor_SMD:R_0805_2012Metric
- R50, R51: renamed from R?; footprint (none) -> Resistor_SMD:R_0805_2012Metric
Connections:
- net RX: now also D11.2 (A)
- net TX: now also D10.2 (A)
- net at R50.1: now also D11.1 (K)
- net at R51.2: now also D10.1 (K)
Changed lines of the file:
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@@
   (symbol (lib_id "Device:R_Small") (at 31.115 49.53 270) (unit 1)
     (in_bom yes) (on_board yes)
-    (property "Reference" "R?" (id 0) (at 31.115 47.625 90))
+    (property "Reference" "R50" (id 0) (at 31.115 47.625 90))
     (property "Value" "1k" (id 1) (at 31.115 45.72 90))
-    (property "Footprint" "" (id 2) (at 31.115 49.53 0)
+    (property "Footprint" "Resistor_SMD:R_0805_2012Metric" (id 2) (at 31.115 49.53 0)
       (effects (font (size 1.27 1.27)) hide)
     )
@@
   (symbol (lib_id "power:+5V") (at 53.34 31.115 0) (unit 1)
     (in_bom yes) (on_board yes) (fields_autoplaced)
-    (property "Reference" "#PWR?" (id 0) (at 53.34 34.925 0)
+    (property "Reference" "#PWR0144" (id 0) (at 53.34 34.925 0)
       (effects (font (size 1.27 1.27)) hide)
     )
@@
     (property "Reference" "J50" (id 0) (at 28.575 23.656 90))
     (property "Value" "HC-05" (id 1) (at 28.575 26.1929 90))
-    (property "Footprint" "" (id 2) (at 34.29 29.845 0)
+    (property "Footprint" "CustomFootprints:HC-05" (id 2) (at 34.29 29.845 0)
       (effects (font (size 1.27 1.27)) hide)
     )
@@
     (pin "6")
   )
-  (symbol (lib_id "Device:D_Small") (at 43.18 52.07 0) (unit 1)
-    (in_bom yes) (on_board yes)
-    (property "Reference" "D11" (id 0) (at 43.18 54.61 0))
-    (property "Value" "D_Small" (id 1) (at 43.18 56.515 0))
-    (property "Footprint" "" (id 2) (at 43.18 52.07 90)
-      (effects (font (size 1.27 1.27)) hide)
-    )
-    (property "Datasheet" "~" (id 3) (at 43.18 52.07 90)
-      (effects (font (size 1.27 1.27)) hide)
-    )
-    (pin "1")
-    (pin "2")
-  )
   (symbol (lib_id "Device:R_Small") (at 43.18 38.735 270) (unit 1)
     (in_bom yes) (on_board yes)
     (property "Reference" "R40" (id 0) (at 43.18 40.64 90))
     (property "Value" "100r" (id 1) (at 43.18 36.8355 90))
-    (property "Footprint" "" (id 2) (at 43.18 38.735 0)
+    (property "Footprint" "Resistor_SMD:R_0805_2012Metric" (id 2) (at 43.18 38.735 0)
       (effects (font (size 1.27 1.27)) hide)
     )
@@
     (pin "2")
   )
+  (symbol (lib_id "Device:LED_Small") (at 43.18 49.53 0) (unit 1)
+    (in_bom yes) (on_board yes)
+    (property "Reference" "D11" (id 0) (at 43.2435 44.1792 0))
+    (property "Value" "LED_Small" (id 1) (at 43.2435 46.7161 0))
+    (property "Footprint" "Diode_SMD:D_0805_2012Metric" (id 2) (at 43.18 49.53 90)
+      (effects (font (size 1.27 1.27)) hide)
+    )
+    (property "Datasheet" "~" (id 3) (at 43.18 49.53 90)
+      (effects (font (size 1.27 1.27)) hide)
+    )
+    (pin "1")
+    (pin "2")
+  )
   (symbol (lib_id "power:GND") (at 24.13 52.705 0) (unit 1)
     (in_bom yes) (on_board yes) (fields_autoplaced)
-    (property "Reference" "#PWR?" (id 0) (at 24.13 59.055 0)
+    (property "Reference" "#PWR0145" (id 0) (at 24.13 59.055 0)
       (effects (font (size 1.27 1.27)) hide)
     )
@@
     (pin "1")
   )
-  (symbol (lib_id "Device:D_Small") (at 43.18 49.53 0) (unit 1)
-    (in_bom yes) (on_board yes)
-    (property "Reference" "D10" (id 0) (at 43.18 45.72 0))
-    (property "Value" "D_Small" (id 1) (at 43.18 47.3511 0))
-    (property "Footprint" "" (id 2) (at 43.18 49.53 90)
-      (effects (font (size 1.27 1.27)) hide)
-    )
-    (property "Datasheet" "~" (id 3) (at 43.18 49.53 90)
-      (effects (font (size 1.27 1.27)) hide)
-    )
-    (pin "1")
-    (pin "2")
-  )
   (symbol (lib_id "power:GND") (at 53.34 33.655 0) (unit 1)
     (in_bom yes) (on_board yes) (fields_autoplaced)
-    (property "Reference" "#PWR?" (id 0) (at 53.34 40.005 0)
+    (property "Reference" "#PWR0146" (id 0) (at 53.34 40.005 0)
       (effects (font (size 1.27 1.27)) hide)
     )
@@
   (symbol (lib_id "Device:R_Small") (at 31.115 52.07 90) (unit 1)
     (in_bom yes) (on_board yes)
-    (property "Reference" "R?" (id 0) (at 31.115 53.975 90))
+    (property "Reference" "R51" (id 0) (at 31.115 53.975 90))
     (property "Value" "1k" (id 1) (at 31.115 55.88 90))
-    (property "Footprint" "" (id 2) (at 31.115 52.07 0)
+    (property "Footprint" "Resistor_SMD:R_0805_2012Metric" (id 2) (at 31.115 52.07 0)
       (effects (font (size 1.27 1.27)) hide)
     )
@@
       (effects (font (size 1.27 1.27)) hide)
     )
+    (pin "1")
+    (pin "2")
+  )
+  (symbol (lib_id "Device:LED_Small") (at 43.18 52.07 0) (unit 1)
+    (in_bom yes) (on_board yes)
+    (property "Reference" "D10" (id 0) (at 43.18 53.975 0))
+    (property "Value" "LED_Small" (id 1) (at 43.18 55.88 0))
+    (property "Footprint" "Diode_SMD:D_0805_2012Metric" (id 2) (at 43.18 52.07 90)
+      (effects (font (size 1.27 1.27)) hide)
+    )
+    (property "Datasheet" "~" (id 3) (at 43.18 52.07 90)
+      (effects (font (size 1.27 1.27)) hide)
+    )
