File: PowerFixes.kicad_sch (KiCad schematic)
At the start: 4 parts

Commit message: Merged in everyone's schematic changes
Parts:
- removed SW?: SW_DPDT_x2, symbol Switch:SW_DPDT_x2
- added D1: LED_Small, symbol Device:LED_Small
- added R30: 1k, symbol Device:R_Small
- added SW1: SW_SPDT, symbol Switch:SW_SPDT
- gave numbers to parts that had none: 2
Connections:
- net +5V: now also R30.2, SW1.2 (B)
- net VUSB: now also SW1.1 (A)
- net at C31.2, U?.1 (OUT): now also SW1.3 (C)
- new net: D1.2 (A), R30.1
- new net GND: D1.1 (K)
Changed lines of the file:
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@@
+    (stroke (width 0) (type default) (color 0 0 0 0))
+  )
+  (wire (pts (xy 36.83 66.675) (xy 38.735 66.675))
     (stroke (width 0) (type default) (color 0 0 0 0))
   )
@@
     (stroke (width 0) (type default) (color 0 0 0 0))
   )
+  (wire (pts (xy 29.845 66.675) (xy 31.75 66.675))
+    (stroke (width 0) (type default) (color 0 0 0 0))
+  )
   (text "ESR Must Be <20 ohms for these capacitors" (at 16.51 19.05 0)
     (effects (font (size 1.27 1.27)) (justify left bottom))
@@
     )
   )
-  (symbol (lib_id "Switch:SW_DPDT_x2") (at 37.465 53.975 0) (unit 1)
+  (symbol (lib_id "Device:LED_Small") (at 27.305 66.675 0) (unit 1)
     (in_bom yes) (on_board yes) (fields_autoplaced)
-    (property "Reference" "SW?" (id 0) (at 37.465 47.3542 0))
-    (property "Value" "SW_DPDT_x2" (id 1) (at 37.465 49.8911 0))
-    (property "Footprint" "" (id 2) (at 37.465 53.975 0)
+    (property "Reference" "D1" (id 0) (at 27.3685 61.3242 0))
+    (property "Value" "LED_Small" (id 1) (at 27.3685 63.8611 0))
+    (property "Footprint" "" (id 2) (at 27.305 66.675 90)
       (effects (font (size 1.27 1.27)) hide)
     )
-    (property "Datasheet" "~" (id 3) (at 37.465 53.975 0)
+    (property "Datasheet" "~" (id 3) (at 27.305 66.675 90)
       (effects (font (size 1.27 1.27)) hide)
     )
     (pin "1")
     (pin "2")
-    (pin "3")
-    (pin "4")
-    (pin "5")
-    (pin "6")
   )
   (symbol (lib_id "Device:C_Small") (at 33.655 25.4 90) (unit 1)
     (in_bom yes) (on_board yes)
-    (property "Reference" "C?" (id 0) (at 33.6613 20.1381 90))
+    (property "Reference" "C30" (id 0) (at 33.6613 20.1381 90))
     (property "Value" "10uF" (id 1) (at 33.6613 22.675 90))
     (property "Footprint" "" (id 2) (at 33.655 25.4 0)
@@
   (symbol (lib_id "Device:C_Small") (at 42.545 25.4 90) (unit 1)
     (in_bom yes) (on_board yes) (fields_autoplaced)
-    (property "Reference" "C?" (id 0) (at 42.5513 20.1381 90))
+    (property "Reference" "C31" (id 0) (at 42.5513 20.1381 90))
     (property "Value" "22uF" (id 1) (at 42.5513 22.675 90))
     (property "Footprint" "" (id 2) (at 42.545 25.4 0)
@@
     (pin "1")
   )
+  (symbol (lib_id "power:+5V") (at 38.735 66.675 0) (unit 1)
+    (in_bom yes) (on_board yes) (fields_autoplaced)
+    (property "Reference" "#PWR?" (id 0) (at 38.735 70.485 0)
+      (effects (font (size 1.27 1.27)) hide)
+    )
+    (property "Value" "+5V" (id 1) (at 38.735 63.0992 0))
+    (property "Footprint" "" (id 2) (at 38.735 66.675 0)
+      (effects (font (size 1.27 1.27)) hide)
+    )
+    (property "Datasheet" "" (id 3) (at 38.735 66.675 0)
+      (effects (font (size 1.27 1.27)) hide)
+    )
+    (pin "1")
+  )
+  (symbol (lib_id "Device:R_Small") (at 34.29 66.675 90) (unit 1)
+    (in_bom yes) (on_board yes)
+    (property "Reference" "R30" (id 0) (at 34.29 68.58 90))
+    (property "Value" "1k" (id 1) (at 34.29 71.1169 90))
+    (property "Footprint" "" (id 2) (at 34.29 66.675 0)
+      (effects (font (size 1.27 1.27)) hide)
+    )
+    (property "Datasheet" "~" (id 3) (at 34.29 66.675 0)
+      (effects (font (size 1.27 1.27)) hide)
+    )
+    (pin "1")
+    (pin "2")
+  )
+  (symbol (lib_id "power:GND") (at 24.765 66.675 0) (unit 1)
+    (in_bom yes) (on_board yes) (fields_autoplaced)
+    (property "Reference" "#PWR?" (id 0) (at 24.765 73.025 0)
+      (effects (font (size 1.27 1.27)) hide)
+    )
+    (property "Value" "GND" (id 1) (at 24.765 71.1184 0))
+    (property "Footprint" "" (id 2) (at 24.765 66.675 0)
+      (effects (font (size 1.27 1.27)) hide)
+    )
+    (property "Datasheet" "" (id 3) (at 24.765 66.675 0)
+      (effects (font (size 1.27 1.27)) hide)
+    )
+    (pin "1")
+  )
+  (symbol (lib_id "Switch:SW_SPDT") (at 37.465 53.975 0) (unit 1)
+    (in_bom yes) (on_board yes) (fields_autoplaced)
+    (property "Reference" "SW1" (id 0) (at 37.465 47.3542 0))
+    (property "Value" "SW_SPDT" (id 1) (at 37.465 49.8911 0))
+    (property "Footprint" "" (id 2) (at 37.465 53.975 0)
+      (effects (font (size 1.27 1.27)) hide)
+    )
+    (property "Datasheet" "~" (id 3) (at 37.465 53.975 0)
+      (effects (font (size 1.27 1.27)) hide)
+    )
+    (pin "1")
+    (pin "2")
+    (pin "3")
+  )
   (symbol (lib_id "power:+8V") (at 27.94 25.4 0) (unit 1)

Commit message: Finishing touches (associating footprints) to schematic
Parts:
- removed SW1: SW_SPDT, symbol Switch:SW_SPDT
- added SW10: L103011MS02Q, CustomFootprints:L103011MS02Q, symbol CustomSymbols:L103011MS02Q
- C30, C31: footprint (none) -> Capacitor_SMD:C_0805_2012Metric
- D1: footprint (none) -> Diode_SMD:D_0805_2012Metric
- R30: footprint (none) -> Resistor_SMD:R_0805_2012Metric
- gave numbers to parts that had none: 1
Connections:
- net +5V: now also SW10.3 (COM_2)
- net VUSB: now also SW10.2 (COM_1)
- net at C31.2, U30.1 (OUT): now also SW10.4 (NO_2)
- no-connect marks 0 -> 1
Changed lines of the file:
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@@
   (junction (at 38.1 25.4) (diameter 0) (color 0 0 0 0)
   )
+  (no_connect (at 55.245 58.42))
   (wire (pts (xy 30.48 25.4) (xy 30.48 33.02))
     (stroke (width 0) (type default) (color 0 0 0 0))
@@
     (stroke (width 0) (type default) (color 0 0 0 0))
   )
-  (wire (pts (xy 28.575 53.975) (xy 32.385 53.975))
+  (wire (pts (xy 48.26 53.34) (xy 55.245 53.34))
+    (stroke (width 0) (type default) (color 0 0 0 0))
+  )
+  (wire (pts (xy 55.245 50.8) (xy 51.435 50.8))
     (stroke (width 0) (type default) (color 0 0 0 0))
   )
@@
     (stroke (width 0) (type default) (color 0 0 0 0))
   )
+  (wire (pts (xy 51.435 50.8) (xy 51.435 33.02))
+    (stroke (width 0) (type default) (color 0 0 0 0))
+  )
   (wire (pts (xy 45.72 33.02) (xy 51.435 33.02))
     (stroke (width 0) (type default) (color 0 0 0 0))
   )
   (wire (pts (xy 45.72 25.4) (xy 45.72 33.02))
-    (stroke (width 0) (type default) (color 0 0 0 0))
-  )
-  (wire (pts (xy 51.435 56.515) (xy 42.545 56.515))
-    (stroke (width 0) (type default) (color 0 0 0 0))
-  )
-  (wire (pts (xy 51.435 33.02) (xy 51.435 56.515))
     (stroke (width 0) (type default) (color 0 0 0 0))
   )
@@
     (effects (font (size 1.27 1.27)) (justify left bottom))
   )
-  (global_label "VUSB" (shape input) (at 42.545 51.435 0) (fields_autoplaced)
-    (effects (font (size 1.27 1.27)) (justify left))
-    (property "Intersheet References" "${INTERSHEET_REFS}" (id 0) (at 49.8567 51.3556 0)
-      (effects (font (size 1.27 1.27)) (justify left) hide)
-    )
+  (global_label "VUSB" (shape input) (at 55.245 55.88 180) (fields_autoplaced)
+    (effects (font (size 1.27 1.27)) (justify right))
+    (property "Intersheet References" "${INTERSHEET_REFS}" (id 0) (at 47.9333 55.9594 0)
+      (effects (font (size 1.27 1.27)) (justify right) hide)
+    )
+  )
+  (symbol (lib_id "CustomSymbols:L103011MS02Q") (at 55.245 50.8 0) (unit 1)
+    (in_bom yes) (on_board yes) (fields_autoplaced)
+    (property "Reference" "SW10" (id 0) (at 76.2762 53.7753 0)
+      (effects (font (size 1.27 1.27)) (justify left))
+    )
+    (property "Value" "L103011MS02Q" (id 1) (at 76.2762 56.3122 0)
+      (effects (font (size 1.27 1.27)) (justify left))
+    )
+    (property "Footprint" "CustomFootprints:L103011MS02Q" (id 2) (at 76.835 48.26 0)
+      (effects (font (size 1.27 1.27)) (justify left) hide)
+    )
+    (property "Datasheet" "https://www.ckswitches.com/media/1423/l.pdf" (id 3) (at 76.835 50.8 0)
+      (effects (font (size 1.27 1.27)) (justify left) hide)
+    )
+    (property "Description" "Slide Switches Slide" (id 4) (at 76.835 53.34 0)
+      (effects (font (size 1.27 1.27)) (justify left) hide)
+    )
+    (property "Height" "14.17" (id 5) (at 76.835 55.88 0)
+      (effects (font (size 1.27 1.27)) (justify left) hide)
+    )
+    (property "Mouser Part Number" "611-L103011MS02Q" (id 6) (at 76.835 58.42 0)
+      (effects (font (size 1.27 1.27)) (justify left) hide)
+    )
+    (property "Mouser Price/Stock" "https://www.mouser.co.uk/ProductDetail/CK/L103011MS02Q?qs=LgMIjt8LuD%252BHRziNfkYfcQ%3D%3D" (id 7) (at 76.835 60.96 0)
+      (effects (font (size 1.27 1.27)) (justify left) hide)
+    )
+    (property "Manufacturer_Name" "C & K COMPONENTS" (id 8) (at 76.835 63.5 0)
+      (effects (font (size 1.27 1.27)) (justify left) hide)
+    )
+    (property "Manufacturer_Part_Number" "L103011MS02Q" (id 9) (at 76.835 66.04 0)
+      (effects (font (size 1.27 1.27)) (justify left) hide)
+    )
+    (pin "1")
+    (pin "2")
+    (pin "3")
+    (pin "4")
   )
   (symbol (lib_id "Device:LED_Small") (at 27.305 66.675 0) (unit 1)
@@
     (property "Reference" "D1" (id 0) (at 27.3685 61.3242 0))
     (property "Value" "LED_Small" (id 1) (at 27.3685 63.8611 0))
-    (property "Footprint" "" (id 2) (at 27.305 66.675 90)
+    (property "Footprint" "Diode_SMD:D_0805_2012Metric" (id 2) (at 27.305 66.675 90)
       (effects (font (size 1.27 1.27)) hide)
     )
@@
     (property "Reference" "C30" (id 0) (at 33.6613 20.1381 90))
     (property "Value" "10uF" (id 1) (at 33.6613 22.675 90))
-    (property "Footprint" "" (id 2) (at 33.655 25.4 0)
+    (property "Footprint" "Capacitor_SMD:C_0805_2012Metric" (id 2) (at 33.655 25.4 0)
       (effects (font (size 1.27 1.27)) hide)
     )
@@
     (property "Reference" "C31" (id 0) (at 42.5513 20.1381 90))
     (property "Value" "22uF" (id 1) (at 42.5513 22.675 90))
-    (property "Footprint" "" (id 2) (at 42.545 25.4 0)
+    (property "Footprint" "Capacitor_SMD:C_0805_2012Metric" (id 2) (at 42.545 25.4 0)
       (effects (font (size 1.27 1.27)) hide)
     )
@@
   (symbol (lib_id "Regulator_Linear:LT1175-5_SOT223") (at 38.1 33.02 0) (unit 1)
     (in_bom yes) (on_board yes) (fields_autoplaced)
-    (property "Reference" "U?" (id 0) (at 38.1 36.9554 0))
+    (property "Reference" "U30" (id 0) (at 38.1 36.9554 0))
     (property "Value" "LT1175-5_SOT223" (id 1) (at 38.1 39.4923 0))
     (property "Footprint" "Package_TO_SOT_SMD:SOT-223-3_TabPin2" (id 2) (at 38.1 38.1 0)
@@
     (pin "3")
   )
-  (symbol (lib_id "power:+5V") (at 28.575 53.975 0) (unit 1)
-    (in_bom yes) (on_board yes) (fields_autoplaced)
-    (property "Reference" "#PWR?" (id 0) (at 28.575 57.785 0)
-      (effects (font (size 1.27 1.27)) hide)
-    )
-    (property "Value" "+5V" (id 1) (at 28.575 50.3992 0))
-    (property "Footprint" "" (id 2) (at 28.575 53.975 0)
-      (effects (font (size 1.27 1.27)) hide)
-    )
-    (property "Datasheet" "" (id 3) (at 28.575 53.975 0)
+  (symbol (lib_id "power:+5V") (at 48.26 53.34 0) (unit 1)
+    (in_bom yes) (on_board yes) (fields_autoplaced)
+    (property "Reference" "#PWR0150" (id 0) (at 48.26 57.15 0)
+      (effects (font (size 1.27 1.27)) hide)
+    )
+    (property "Value" "+5V" (id 1) (at 48.26 49.7642 0))
+    (property "Footprint" "" (id 2) (at 48.26 53.34 0)
+      (effects (font (size 1.27 1.27)) hide)
+    )
+    (property "Datasheet" "" (id 3) (at 48.26 53.34 0)
       (effects (font (size 1.27 1.27)) hide)
     )
@@
   (symbol (lib_id "power:+5V") (at 38.735 66.675 0) (unit 1)
     (in_bom yes) (on_board yes) (fields_autoplaced)
-    (property "Reference" "#PWR?" (id 0) (at 38.735 70.485 0)
+    (property "Reference" "#PWR0149" (id 0) (at 38.735 70.485 0)
       (effects (font (size 1.27 1.27)) hide)
     )
@@
     (property "Reference" "R30" (id 0) (at 34.29 68.58 90))
     (property "Value" "1k" (id 1) (at 34.29 71.1169 90))
-    (property "Footprint" "" (id 2) (at 34.29 66.675 0)
+    (property "Footprint" "Resistor_SMD:R_0805_2012Metric" (id 2) (at 34.29 66.675 0)
       (effects (font (size 1.27 1.27)) hide)
     )
@@
   (symbol (lib_id "power:GND") (at 24.765 66.675 0) (unit 1)
     (in_bom yes) (on_board yes) (fields_autoplaced)
-    (property "Reference" "#PWR?" (id 0) (at 24.765 73.025 0)
+    (property "Reference" "#PWR0148" (id 0) (at 24.765 73.025 0)
       (effects (font (size 1.27 1.27)) hide)
     )
@@
     (pin "1")
   )
-  (symbol (lib_id "Switch:SW_SPDT") (at 37.465 53.975 0) (unit 1)
-    (in_bom yes) (on_board yes) (fields_autoplaced)
-    (property "Reference" "SW1" (id 0) (at 37.465 47.3542 0))
-    (property "Value" "SW_SPDT" (id 1) (at 37.465 49.8911 0))
-    (property "Footprint" "" (id 2) (at 37.465 53.975 0)
-      (effects (font (size 1.27 1.27)) hide)
-    )
-    (property "Datasheet" "~" (id 3) (at 37.465 53.975 0)
-      (effects (font (size 1.27 1.27)) hide)
-    )
-    (pin "1")
-    (pin "2")
-    (pin "3")
-  )
   (symbol (lib_id "power:+8V") (at 27.94 25.4 0) (unit 1)
     (in_bom yes) (on_board yes) (fields_autoplaced)
-    (property "Reference" "#PWR?" (id 0) (at 27.94 29.21 0)
-      (effects (font (size 1.27 1.27)) hide)
-    )
+    (property "Reference" "#PWR0147" (id 0) (at 27.94 29.21 0)
+      (effects (font (size 1.27 1.27)) hide)
+    )

Commit message: Finishing touches 2 (extra test points)
Connections:
- net VREG: now reaches C31.2, SW10.4 (NO_2), U30.1 (OUT)
Changed lines of the file:
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@@
     (effects (font (size 1.27 1.27)) (justify left bottom))
+  )
+  (global_label "VREG" (shape input) (at 51.435 33.02 0) (fields_autoplaced)
+    (effects (font (size 1.27 1.27)) (justify left))
+    (property "Intersheet References" "${INTERSHEET_REFS}" (id 0) (at 58.6257 32.9406 0)
+      (effects (font (size 1.27 1.27)) (justify left) hide)
+    )
   )
   (global_label "VUSB" (shape input) (at 55.245 55.88 180) (fields_autoplaced)

Commit message: Pushing PCB
Parts:
- removed U30: LT1175-5_SOT223, Package_TO_SOT_SMD:SOT-223-3_TabPin2, symbol Regulator_Linear:LT1175-5_SOT223
- added U30: AZ1117I-5.0, Package_TO_SOT_SMD:SOT-223-3_TabPin2, symbol Regulator_Linear:NCP1117-12_SOT223
Connections:
- net +8V: now also U30.3 (VI)
- net GND: now also C30.2, C31.1, U30.1 (GND)
- net VREG: now also U30.2 (VO)
Changed lines of the file:
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@@
+    (stroke (width 0) (type default) (color 0 0 0 0))
+  )
+  (wire (pts (xy 38.1 25.4) (xy 38.1 21.59))
     (stroke (width 0) (type default) (color 0 0 0 0))
   )
   (wire (pts (xy 30.48 25.4) (xy 31.115 25.4))
+    (stroke (width 0) (type default) (color 0 0 0 0))
+  )
+  (wire (pts (xy 38.1 21.59) (xy 50.8 21.59))
     (stroke (width 0) (type default) (color 0 0 0 0))
   )
@@
     (pin "2")
   )
-  (symbol (lib_id "Regulator_Linear:LT1175-5_SOT223") (at 38.1 33.02 0) (unit 1)
-    (in_bom yes) (on_board yes) (fields_autoplaced)
-    (property "Reference" "U30" (id 0) (at 38.1 36.9554 0))
-    (property "Value" "LT1175-5_SOT223" (id 1) (at 38.1 39.4923 0))
-    (property "Footprint" "Package_TO_SOT_SMD:SOT-223-3_TabPin2" (id 2) (at 38.1 38.1 0)
-      (effects (font (size 1.27 1.27)) hide)
-    )
-    (property "Datasheet" "https://www.analog.com/media/en/technical-documentation/data-sheets/1175ff.pdf" (id 3) (at 38.735 33.02 0)
-      (effects (font (size 1.27 1.27)) hide)
-    )
-    (pin "1")
-    (pin "2")
-    (pin "3")
-  )
   (symbol (lib_id "power:+5V") (at 48.26 53.34 0) (unit 1)
     (in_bom yes) (on_board yes) (fields_autoplaced)
@@
     (pin "1")
   )
+  (symbol (lib_id "power:GND") (at 50.8 21.59 0) (unit 1)
+    (in_bom yes) (on_board yes) (fields_autoplaced)
+    (property "Reference" "#PWR0152" (id 0) (at 50.8 27.94 0)
+      (effects (font (size 1.27 1.27)) hide)
+    )
+    (property "Value" "GND" (id 1) (at 50.8 26.0334 0))
+    (property "Footprint" "" (id 2) (at 50.8 21.59 0)
+      (effects (font (size 1.27 1.27)) hide)
+    )
+    (property "Datasheet" "" (id 3) (at 50.8 21.59 0)
+      (effects (font (size 1.27 1.27)) hide)
+    )
+    (pin "1")
+  )
+  (symbol (lib_id "Regulator_Linear:NCP1117-12_SOT223") (at 38.1 33.02 0) (mirror x) (unit 1)
+    (in_bom yes) (on_board yes) (fields_autoplaced)
+    (property "Reference" "U30" (id 0) (at 38.1 36.9554 0))
+    (property "Value" "AZ1117I-5.0" (id 1) (at 38.1 39.4923 0))
+    (property "Footprint" "Package_TO_SOT_SMD:SOT-223-3_TabPin2" (id 2) (at 38.1 38.1 0)
+      (effects (font (size 1.27 1.27)) hide)
+    )
+    (property "Datasheet" "http://www.onsemi.com/pub_link/Collateral/NCP1117-D.PDF" (id 3) (at 40.64 26.67 0)
+      (effects (font (size 1.27 1.27)) hide)
+    )
+    (pin "1")
+    (pin "2")
+    (pin "3")
+  )
   (symbol (lib_id "Device:R_Small") (at 34.29 66.675 90) (unit 1)
